File: PWR-MGR-PCB/PWR-MGR-PCB.kicad_pcb (KiCad board)
At the start: 2 copper layers, 23 parts, among them J1 USB_C_Receptacle_USB2.0_14P, J2 Battery_1x2, J3 Conn_01x01_Pin, J4 Conn_01x01_Pin, J5 Conn_01x01_Pin, J6 Conn_01x01_Pin, U1 USBLC6-2SC6, U2 TLV75533PDBV, U3 BQ24074RGT

Commit message: Start layout
Parts:
- moved J1 26.8 mm to (152.4, 106.7)
- moved J2 18.1 mm to (170.7, 87.3)
- moved R2 6.51 mm to (133.0, 75.4)
- moved R3 6.51 mm to (133.0, 78.3)
- moved R4 6.51 mm to (133.0, 81.3)
- moved R5 6.51 mm to (133.0, 84.2)
- moved R8 6.51 mm to (133.0, 90.1)
- moved R1 6.51 mm to (133.0, 72.4)
- moved R6 6.51 mm to (133.0, 87.2)
- moved C1 5.36 mm to (146.7, 80.8)
- moved J3 5.36 mm to (142.2, 71.6)
- moved J5 5.36 mm to (142.2, 80.8)
- moved C2 5.36 mm to (146.7, 83.8)
- moved J4 5.36 mm to (142.2, 76.2)
- moved J6 5.36 mm to (142.2, 85.4)
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Other:
- board outline added: 50.8 x 45.7 mm
Changed lines of the file:
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@@
 	(footprint "Connector_JST:JST_PH_B2B-PH-K_1x02_P2.00mm_Vertical"
 		(layer "F.Cu")
-		(at 152.625 87.31)
+		(at 170.72 87.31)
 		(descr "JST PH series connector, B2B-PH-K (http://www.jst-mfg.com/product/pdf/eng/ePH.pdf), generated with kicad-footprint-generator")
 		(tags "connector JST PH vertical")
@@
 	(footprint "Resistor_SMD:R_0805_2012Metric"
 		(layer "F.Cu")
-		(at 138.395 84.92)
+		(at 132.9925 81.28)
 		(descr "Resistor SMD 0805 (2012 Metric), square (rectangular) end terminal, IPC-7351 nominal, (Body size source: IPC-SM-782 page 72, https://www.pcb-3d.com/wordpress/wp-content/uploads/ipc-sm-782a_amendment_1_and_2.pdf), generated with kicad-footprint-generator")
 		(tags "resistor")
@@
 	(footprint "Connector_USB:USB_C_Receptacle_GCT_USB4105-xx-A_16P_TopMnt_Horizontal"
 		(layer "F.Cu")
-		(at 151.045 79.88)
+		(at 152.4 106.68)
 		(descr "USB 2.0 Type C Receptacle, GCT, 16P, top mounted, horizontal, 5A: https://gct.co/files/drawings/usb4105.pdf")
 		(tags "USB C Type-C Receptacle SMD USB 2.0 16P 16C USB4105-15-A USB4105-15-A-060 USB4105-15-A-120 USB4105-GF-A USB4105-GF-A-060 USB4105-GF-A-120")
 		(property "Reference" "J1"
-			(at 0 -5.5 0)
+			(at 4.1175 -6.645 0)
 			(unlocked yes)
 			(layer "F.SilkS")
@@
 	(footprint "Capacitor_SMD:C_0805_2012Metric"
 		(layer "F.Cu")
-		(at 147.425 89.1)
+		(at 146.74 83.78)
 		(descr "Capacitor SMD 0805 (2012 Metric), square (rectangular) end terminal, IPC-7351 nominal, (Body size source: IPC-SM-782 page 76, https://www.pcb-3d.com/wordpress/wp-content/uploads/ipc-sm-782a_amendment_1_and_2.pdf, https://docs.google.com/spreadsheets/d/1BsfQQcO9C6DZCsRaXUlFlo91Tg2WpOkGARC1WS5S8t0/edit?usp=sharing), generated with kicad-footprint-generator")
 		(tags "capacitor")
@@
 	(footprint "BQ24074RGTR:QFN50P300X300X100-17N"
 		(layer "F.Cu")
-		(at 157.975 93.775)
+		(at 162.0925 92.63)
 		(property "Reference" "U3"
 			(at -0.165 -3.24 0)
@@
 	(footprint "Package_TO_SOT_SMD:SOT-23-5"
 		(layer "F.Cu")
-		(at 152.225 98.16)
+		(at 156.3425 97.015)
 		(descr "SOT, 5 Pin (JEDEC MO-178 Var AA https://www.jedec.org/document_search?search_api_views_fulltext=MO-178), generated with kicad-footprint-generator ipc_gullwing_generator.py")
 		(tags "SOT TO_SOT_SMD")
@@
 	(footprint "Capacitor_SMD:C_0805_2012Metric"
 		(layer "F.Cu")
-		(at 147.425 98.13)
+		(at 151.5425 96.985)
 		(descr "Capacitor SMD 0805 (2012 Metric), square (rectangular) end terminal, IPC-7351 nominal, (Body size source: IPC-SM-782 page 76, https://www.pcb-3d.com/wordpress/wp-content/uploads/ipc-sm-782a_amendment_1_and_2.pdf, https://docs.google.com/spreadsheets/d/1BsfQQcO9C6DZCsRaXUlFlo91Tg2WpOkGARC1WS5S8t0/edit?usp=sharing), generated with kicad-footprint-generator")
 		(tags "capacitor")
@@
 	(footprint "Connector_PinSocket_2.54mm:PinSocket_1x01_P2.54mm_Vertical"
 		(layer "F.Cu")
-		(at 142.925 90.72)
+		(at 142.24 85.4)
 		(descr "Through hole straight socket strip, 1x01, 2.54mm pitch, single row (from Kicad 4.0.7), script generated")
 		(tags "Through hole socket strip THT 1x01 2.54mm single row")
@@
 		)
 		(property "Value" "Conn_01x01_Pin"
-			(at 0 2.77 0)
+			(at 4.1175 1.625 0)
 			(layer "F.Fab")
 			(effects
@@
 	(footprint "Connector_PinSocket_2.54mm:PinSocket_1x01_P2.54mm_Vertical"
 		(layer "F.Cu")
-		(at 142.925 76.92)
+		(at 142.24 71.6)
 		(descr "Through hole straight socket strip, 1x01, 2.54mm pitch, single row (from Kicad 4.0.7), script generated")
 		(tags "Through hole socket strip THT 1x01 2.54mm single row")
@@
 	(footprint "Resistor_SMD:R_0805_2012Metric"
 		(layer "F.Cu")
-		(at 138.395 87.87)
+		(at 132.9925 84.23)
 		(descr "Resistor SMD 0805 (2012 Metric), square (rectangular) end terminal, IPC-7351 nominal, (Body size source: IPC-SM-782 page 72, https://www.pcb-3d.com/wordpress/wp-content/uploads/ipc-sm-782a_amendment_1_and_2.pdf), generated with kicad-footprint-generator")
 		(tags "resistor")
@@
 	(footprint "LED - SML_D12U1WT86:LED_SML-D12U1WT86"
 		(layer "F.Cu")
-		(at 143.065 96.52)
+		(at 147.1825 95.375)
 		(property "Reference" "D2"
 			(at 0.532 -1.4064 0)
@@
 	(footprint "LED - SML_D12U1WT86:LED_SML-D12U1WT86"
 		(layer "F.Cu")
-		(at 143.065 94.17)
+		(at 147.1825 93.025)
 		(property "Reference" "D1"
 			(at 0.532 -1.4064 0)
@@
 	(footprint "Connector_PinSocket_2.54mm:PinSocket_1x01_P2.54mm_Vertical"
 		(layer "F.Cu")
-		(at 142.925 81.52)
+		(at 142.24 76.2)
 		(descr "Through hole straight socket strip, 1x01, 2.54mm pitch, single row (from Kicad 4.0.7), script generated")
 		(tags "Through hole socket strip THT 1x01 2.54mm single row")
@@
 	(footprint "Resistor_SMD:R_0805_2012Metric"
 		(layer "F.Cu")
-		(at 138.395 93.77)
+		(at 132.9925 90.13)
 		(descr "Resistor SMD 0805 (2012 Metric), square (rectangular) end terminal, IPC-7351 nominal, (Body size source: IPC-SM-782 page 72, https://www.pcb-3d.com/wordpress/wp-content/uploads/ipc-sm-782a_amendment_1_and_2.pdf), generated with kicad-footprint-generator")
 		(tags "resistor")
@@
 	(footprint "Resistor_SMD:R_0805_2012Metric"
 		(layer "F.Cu")
-		(at 138.395 90.82)
+		(at 132.9925 87.18)
 		(descr "Resistor SMD 0805 (2012 Metric), square (rectangular) end terminal, IPC-7351 nominal, (Body size source: IPC-SM-782 page 72, https://www.pcb-3d.com/wordpress/wp-content/uploads/ipc-sm-782a_amendment_1_and_2.pdf), generated with kicad-footprint-generator")
 		(tags "resistor")
@@
 	(footprint "Resistor_SMD:R_0805_2012Metric"
 		(layer "F.Cu")
-		(at 138.395 76.07)
+		(at 132.9925 72.43)
 		(descr "Resistor SMD 0805 (2012 Metric), square (rectangular) end terminal, IPC-7351 nominal, (Body size source: IPC-SM-782 page 72, https://www.pcb-3d.com/wordpress/wp-content/uploads/ipc-sm-782a_amendment_1_and_2.pdf), generated with kicad-footprint-generator")
 		(tags "resistor")
@@
 	(footprint "Package_TO_SOT_SMD:SOT-23-6"
 		(layer "F.Cu")
-		(at 152.225 93.535)
+		(at 156.3425 92.39)
 		(descr "SOT, 6 Pin (JEDEC MO-178 Var AB https://www.jedec.org/document_search?search_api_views_fulltext=MO-178), generated with kicad-footprint-generator ipc_gullwing_generator.py")
 		(tags "SOT TO_SOT_SMD")
@@
 	(footprint "Capacitor_SMD:C_0805_2012Metric"
 		(layer "F.Cu")
-		(at 147.425 92.11)
+		(at 151.5425 90.965)
 		(descr "Capacitor SMD 0805 (2012 Metric), square (rectangular) end terminal, IPC-7351 nominal, (Body size source: IPC-SM-782 page 76, https://www.pcb-3d.com/wordpress/wp-content/uploads/ipc-sm-782a_amendment_1_and_2.pdf, https://docs.google.com/spreadsheets/d/1BsfQQcO9C6DZCsRaXUlFlo91Tg2WpOkGARC1WS5S8t0/edit?usp=sharing), generated with kicad-footprint-generator")
 		(tags "capacitor")
 		(property "Reference" "C3"
-			(at 0 -1.68 0)
+			(at -0.685 -7 0)
 			(layer "F.SilkS")
 			(effects
@@
 	(footprint "Resistor_SMD:R_0805_2012Metric"
 		(layer "F.Cu")
-		(at 138.395 81.97)
+		(at 132.9925 78.33)
 		(descr "Resistor SMD 0805 (2012 Metric), square (rectangular) end terminal, IPC-7351 nominal, (Body size source: IPC-SM-782 page 72, https://www.pcb-3d.com/wordpress/wp-content/uploads/ipc-sm-782a_amendment_1_and_2.pdf), generated with kicad-footprint-generator")
 		(tags "resistor")
@@
 	(footprint "Connector_PinSocket_2.54mm:PinSocket_1x01_P2.54mm_Vertical"
 		(layer "F.Cu")
-		(at 142.925 86.12)
+		(at 142.24 80.8)
 		(descr "Through hole straight socket strip, 1x01, 2.54mm pitch, single row (from Kicad 4.0.7), script generated")
 		(tags "Through hole socket strip THT 1x01 2.54mm single row")
@@
 	(footprint "Capacitor_SMD:C_0805_2012Metric"
 		(layer "F.Cu")
-		(at 147.425 86.09)
+		(at 146.74 80.77)
 		(descr "Capacitor SMD 0805 (2012 Metric), square (rectangular) end terminal, IPC-7351 nominal, (Body size source: IPC-SM-782 page 76, https://www.pcb-3d.com/wordpress/wp-content/uploads/ipc-sm-782a_amendment_1_and_2.pdf, https://docs.google.com/spreadsheets/d/1BsfQQcO9C6DZCsRaXUlFlo91Tg2WpOkGARC1WS5S8t0/edit?usp=sharing), generated with kicad-footprint-generator")
 		(tags "capacitor")
@@
 	(footprint "Resistor_SMD:R_0805_2012Metric"
 		(layer "F.Cu")
-		(at 138.395 79.02)
+		(at 132.9925 75.38)
 		(descr "Resistor SMD 0805 (2012 Metric), square (rectangular) end terminal, IPC-7351 nominal, (Body size source: IPC-SM-782 page 72, https://www.pcb-3d.com/wordpress/wp-content/uploads/ipc-sm-782a_amendment_1_and_2.pdf), generated with kicad-footprint-generator")
 		(tags "resistor")
@@
 	(footprint "Capacitor_SMD:C_0805_2012Metric"
 		(layer "F.Cu")
-		(at 147.425 95.12)
+		(at 151.5425 93.975)
 		(descr "Capacitor SMD 0805 (2012 Metric), square (rectangular) end terminal, IPC-7351 nominal, (Body size source: IPC-SM-782 page 76, https://www.pcb-3d.com/wordpress/wp-content/uploads/ipc-sm-782a_amendment_1_and_2.pdf, https://docs.google.com/spreadsheets/d/1BsfQQcO9C6DZCsRaXUlFlo91Tg2WpOkGARC1WS5S8t0/edit?usp=sharing), generated with kicad-footprint-generator")
 		(tags "capacitor")
@@
 		)
 	)
+	(gr_line
+		(start 127 66.04)
+		(end 127 111.76)
+		(stroke
+			(width 0.05)
+			(type default)
+		)
+		(layer "Edge.Cuts")
+	)
+	(gr_line
+		(start 177.8 66.04)
+		(end 127 66.04)
+		(stroke
+			(width 0.05)
+			(type default)
+		)
+		(layer "Edge.Cuts")
+	)
+	(gr_line
+		(start 127 111.76)
+		(end 177.8 111.76)
+		(stroke
+			(width 0.05)
+			(type default)
+		)
+		(layer "Edge.Cuts")
+	)
+	(gr_line
+		(start 177.8 111.76)
+		(end 177.8 66.04)
+		(stroke
+			(width 0.05)
+			(type default)
+		)
+		(layer "Edge.Cuts")
+	)
 	(embedded_fonts no)

Commit message: Layout PCB
Parts:
- moved J3 32.2 mm to (143.9, 103.8)
- moved R1 31.6 mm to (151.4, 98.1), turned to 90 degrees
- moved R3 28.4 mm to (159.0, 89.8), turned to 180 degrees
- moved R4 28.3 mm to (159.0, 92.4), turned to 180 degrees
- moved R6 27.8 mm to (160.8, 86.2)
- moved R5 27.8 mm to (160.8, 83.5)
- moved R2 27.4 mm to (148.0, 98.3), turned to 90 degrees
- moved J5 27.0 mm to (168.7, 86.0)
- moved U2 18.8 mm to (152.5, 78.6)
- moved J6 16.5 mm to (153.0, 72.9)
- moved D2 15.7 mm to (157.3, 83.4)
- moved C2 14.1 mm to (158.7, 76.5)
- moved R8 13.8 mm to (146.6, 88.4), turned to 180 degrees
- moved D1 12.1 mm to (157.2, 86.2)
- moved U3 9.68 mm to (152.8, 90.1), turned to 90 degrees
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
Commit message: Resize board
Other:
- board size 50.8 x 45.7 mm -> 32 x 45.7 mm
Changed lines of the file:
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@@
 			(unlocked yes)
 			(layer "F.Fab")
+			(hide yes)
 			(effects
 				(font
@@
 			(at 0 2.77 0)
 			(layer "F.Fab")
+			(hide yes)
 			(effects
 				(font
@@
 	)
 	(gr_line
-		(start 127 66.04)
-		(end 127 111.76)
+		(start 141.3256 66.04)
+		(end 141.3256 111.76)
 		(stroke
 			(width 0.05)
@@
 	)
 	(gr_line
-		(start 177.8 66.04)
-		(end 127 66.04)
+		(start 173.3296 66.04)
+		(end 141.3256 66.04)
 		(stroke
 			(width 0.05)
@@
 	)
 	(gr_line
-		(start 127 111.76)
-		(end 177.8 111.76)
+		(start 141.3256 111.76)
+		(end 173.3296 111.76)
 		(stroke
 			(width 0.05)
@@
 	)
 	(gr_line
-		(start 177.8 111.76)
-		(end 177.8 66.04)
+		(start 173.3296 111.76)
+		(end 173.3296 66.04)
 		(stroke
 			(width 0.05)

Commit message: Layout board
Parts:
- moved C4 3.23 mm to (151.7, 81.2)
- moved C1 3.23 mm to (147.2, 74.3)
- moved J6 3.23 mm to (153.3, 69.7)
- moved U2 3.23 mm to (152.7, 75.4)
- moved J4 3.23 mm to (146.7, 80.6)
- moved C2 1.61 mm to (158.5, 74.9)
Changed lines of the file:
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@@
 	(footprint "Capacitor_SMD:C_0805_2012Metric"
 		(layer "F.Cu")
-		(at 158.7453 76.4755)
+		(at 158.5112 74.8792)
 		(descr "Capacitor SMD 0805 (2012 Metric), square (rectangular) end terminal, IPC-7351 nominal, (Body size source: IPC-SM-782 page 76, https://www.pcb-3d.com/wordpress/wp-content/uploads/ipc-sm-782a_amendment_1_and_2.pdf, https://docs.google.com/spreadsheets/d/1BsfQQcO9C6DZCsRaXUlFlo91Tg2WpOkGARC1WS5S8t0/edit?usp=sharing), generated with kicad-footprint-generator")
 		(tags "capacitor")
@@
 	(footprint "Package_TO_SOT_SMD:SOT-23-5"
 		(layer "F.Cu")
-		(at 152.5016 78.5735)
+		(at 152.7247 75.3516)
 		(descr "SOT, 5 Pin (JEDEC MO-178 Var AA https://www.jedec.org/document_search?search_api_views_fulltext=MO-178), generated with kicad-footprint-generator ipc_gullwing_generator.py")
 		(tags "SOT TO_SOT_SMD")
@@
 	(footprint "Connector_PinSocket_2.54mm:PinSocket_1x01_P2.54mm_Vertical"
 		(layer "F.Cu")
-		(at 153.0405 72.9195)
+		(at 153.2636 69.6976)
 		(descr "Through hole straight socket strip, 1x01, 2.54mm pitch, single row (from Kicad 4.0.7), script generated")
 		(tags "Through hole socket strip THT 1x01 2.54mm single row")
@@
 	(footprint "Connector_PinSocket_2.54mm:PinSocket_1x01_P2.54mm_Vertical"
 		(layer "F.Cu")
-		(at 146.5072 83.82)
+		(at 146.7303 80.5981)
 		(descr "Through hole straight socket strip, 1x01, 2.54mm pitch, single row (from Kicad 4.0.7), script generated")
 		(tags "Through hole socket strip THT 1x01 2.54mm single row")
@@
 	(footprint "Capacitor_SMD:C_0805_2012Metric"
 		(layer "F.Cu")
-		(at 146.9597 77.4915 180)
+		(at 147.1828 74.2696 180)
 		(descr "Capacitor SMD 0805 (2012 Metric), square (rectangular) end terminal, IPC-7351 nominal, (Body size source: IPC-SM-782 page 76, https://www.pcb-3d.com/wordpress/wp-content/uploads/ipc-sm-782a_amendment_1_and_2.pdf, https://docs.google.com/spreadsheets/d/1BsfQQcO9C6DZCsRaXUlFlo91Tg2WpOkGARC1WS5S8t0/edit?usp=sharing), generated with kicad-footprint-generator")
 		(tags "capacitor")
@@
 	(footprint "Capacitor_SMD:C_0805_2012Metric"
 		(layer "F.Cu")
-		(at 151.4348 84.3788 180)
+		(at 151.6579 81.1569 180)
 		(descr "Capacitor SMD 0805 (2012 Metric), square (rectangular) end terminal, IPC-7351 nominal, (Body size source: IPC-SM-782 page 76, https://www.pcb-3d.com/wordpress/wp-content/uploads/ipc-sm-782a_amendment_1_and_2.pdf, https://docs.google.com/spreadsheets/d/1BsfQQcO9C6DZCsRaXUlFlo91Tg2WpOkGARC1WS5S8t0/edit?usp=sharing), generated with kicad-footprint-generator")
 		(tags "capacitor")

Commit message: Route board
Parts:
- moved J6 14.5 mm to (164.9, 78.2)
- moved C1 3.27 mm to (147.2, 77.5)
- moved C2 3.27 mm to (158.5, 78.2), turned to -90 degrees
- moved C4 3.27 mm to (151.7, 84.4)
- moved J4 3.27 mm to (146.8, 83.9)
- moved U2 3.27 mm to (152.8, 78.6)
- moved R1 1.36 mm to (152.8, 98.4)
- moved J2 1.25 mm to (168.7, 93.2)
- moved R2 1.22 mm to (149.3, 98.4)
Routing:
- net GND: track 0.00 -> 129.9 mm, vias 0 -> 4
- net VCC_BMS: track 0.00 -> 53.3 mm, vias 0 -> 1
- net VBUS 5V: track 0.00 -> 49.5 mm, vias 0 -> 2
- net /VBATT_TEST: track 0.00 -> 29.0 mm, vias 0 -> 1
- net Net-(J1-CC2): track 0.00 -> 15.2 mm, vias 0 -> 2
- net /USB_CONN_D+: track 0.00 -> 13.8 mm
- net Net-(U3-ILIM): track 0.00 -> 13.2 mm, vias 0 -> 2
- net +3.3V: track 0.00 -> 11.8 mm
- net Net-(J1-CC1): track 0.00 -> 8.33 mm, vias 0 -> 2
- net /USB_CONN_D-: track 0.00 -> 8.31 mm
- net Net-(U3-~{CHG}): track 0.00 -> 6.75 mm
- net Net-(U3-TS): track 0.00 -> 5.95 mm
- net Net-(U3-~{PGOOD}): track 0.00 -> 4.78 mm
- net Net-(U3-ISET): track 0.00 -> 2.56 mm, vias 0 -> 1
- net Net-(D1-PadA): track 0.00 -> 1.87 mm
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Other:
- board size 32 x 45.7 mm -> 32 x 37.4 mm

Commit message: Reroute board
Parts:
- J1: value USB_C_Receptacle_USB2.0_14P -> USB_C_Receptacle_USB2.0_16P
- moved R1 10.4 mm to (163.0, 100.2), turned to 0 degrees
- moved J6 3.71 mm to (168.7, 78.2)
- moved J1 2.95 mm to (155.2, 107.6)
- moved U1 2.92 mm to (155.4, 99.1)
- moved J5 2.18 mm to (168.7, 83.8)
- moved R2 1.75 mm to (149.8, 100.1), turned to 180 degrees
- turned U3 to 180 degrees
Connections:
- J1 pad A8: (no net) -> unconnected-(J1-SBU1-PadA8)
- J1 pad B8: (no net) -> unconnected-(J1-SBU2-PadB8)
Routing:
- net GND: track 129.9 -> 113.3 mm, vias 4 -> 0
- net Net-(U3-TS): track 5.95 -> 18.6 mm, vias 0 -> 2
- net /USB_CONN_D+: track 13.8 -> 6.71 mm
- net VCC_BMS: track 53.3 -> 47.5 mm, vias 1 -> 0
- net Net-(U3-ILIM): track 13.2 -> 18.0 mm
- net /VBATT_TEST: track 29.0 -> 33.6 mm, vias 1 -> 2
- net Net-(U3-~{CHG}): track 6.75 -> 11.0 mm, vias 0 -> 2
- net Net-(J1-CC2): track 15.2 -> 11.1 mm, vias 2 -> 0
- net Net-(U3-~{PGOOD}): track 4.78 -> 8.51 mm, vias 0 -> 2
- net +3.3V: track 11.8 -> 15.4 mm
- net Net-(U3-ISET): track 2.56 -> 5.54 mm, vias 1 -> 0
- net VBUS 5V: track 49.5 -> 52.2 mm, vias 2 -> 1
- net /USB_CONN_D-: track 8.31 -> 5.70 mm
- net Net-(J1-CC1): track 8.33 -> 10.9 mm, vias 2 -> 0
