File: PWR-MGR-PCB/output.kicad_sch (KiCad schematic)
At the start: 6 parts, among them J1 Conn_01x02_Pin, J5 Conn_01x02_Pin

Commit message: Finish USB data routing, connect VBUS to BQ2407
Parts:
- J1: footprint Connector_JST:JST_XH_B2B-XH-A_1x02_P2.50mm_Vertical -> Connector_PinSocket_1.00mm:PinSocket_1x02_P1.00mm_Vertical
- J5: footprint Connector_PinHeader_1.00mm:PinHeader_1x02_P1.00mm_Vertical_SMD_Pin1Right -> Connector_PinSocket_1.00mm:PinSocket_1x02_P1.00mm_Vertical
Changed lines of the file:
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@@
 			)
 		)
-		(property "Footprint" "Connector_JST:JST_XH_B2B-XH-A_1x02_P2.50mm_Vertical"
+		(property "Footprint" "Connector_PinSocket_1.00mm:PinSocket_1x02_P1.00mm_Vertical"
 			(at 173.99 81.28 0)
 			(effects
@@
 			)
 		)
-		(property "Footprint" "Connector_PinHeader_1.00mm:PinHeader_1x02_P1.00mm_Vertical_SMD_Pin1Right"
+		(property "Footprint" "Connector_PinSocket_1.00mm:PinSocket_1x02_P1.00mm_Vertical"
 			(at 114.3 80.01 0)
 			(effects

Commit message: Change zone connection types, change connectors, add zones for buck boost converter
Parts:
- J1: footprint Connector_PinSocket_1.00mm:PinSocket_1x02_P1.00mm_Vertical -> Connector_JST:JST_XH_B2B-XH-A_1x02_P2.50mm_Vertical
- J5: footprint Connector_PinSocket_1.00mm:PinSocket_1x02_P1.00mm_Vertical -> Connector_PinHeader_2.00mm:PinHeader_1x02_P2.00mm_Vertical
Changed lines of the file:
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@@
 			)
 		)
-		(property "Footprint" "Connector_PinSocket_1.00mm:PinSocket_1x02_P1.00mm_Vertical"
+		(property "Footprint" "Connector_JST:JST_XH_B2B-XH-A_1x02_P2.50mm_Vertical"
 			(at 173.99 81.28 0)
 			(effects
@@
 			)
 		)
-		(property "Footprint" "Connector_PinSocket_1.00mm:PinSocket_1x02_P1.00mm_Vertical"
+		(property "Footprint" "Connector_PinHeader_2.00mm:PinHeader_1x02_P2.00mm_Vertical"
 			(at 114.3 80.01 0)
 			(effects

Commit message: Add MPNs and generate DRL file
Parts:
- J1: Manufacturer Part Number (none) -> B2B-XH-A
- J5: Manufacturer Part Number (none) -> TMM-102-02-T-S
Changed lines of the file:
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@@
+			)
+		)
+		(property "Manufacturer Part Number" ""
+			(at 116.84 105.41 0)
+			(effects
+				(font
+					(size 1.27 1.27)
+				)
+				(hide yes)
 			)
 		)
@@
 			)
 		)
+		(property "Manufacturer Part Number" " B2B-XH-A"
+			(at 173.99 81.28 0)
+			(effects
+				(font
+					(size 1.27 1.27)
+				)
+				(hide yes)
+			)
+		)
 		(pin "1"
 		)
@@
 			)
 		)
+		(property "Manufacturer Part Number" ""
+			(at 92.71 111.76 0)
+			(effects
+				(font
+					(size 1.27 1.27)
+				)
+				(hide yes)
+			)
+		)
 		(instances
 			(project "PWR-MGR-PCB"
@@
 			)
 		)
+		(property "Manufacturer Part Number" ""
+			(at 116.84 111.76 0)
+			(effects
+				(font
+					(size 1.27 1.27)
+				)
+				(hide yes)
+			)
+		)
 		(instances
 			(project "PWR-MGR-PCB"
@@
 			)
 		)
+		(property "Manufacturer Part Number" "TMM-102-02-T-S"
+			(at 114.3 80.01 0)
+			(effects
+				(font
+					(size 1.27 1.27)
+				)
+				(hide yes)
+			)
+		)
 		(pin "1"
 		)
@@
 			(at 92.71 105.41 0)
 			(effects
+				(font
+					(size 1.27 1.27)
+				)
+				(hide yes)
+			)
+		)
+		(property "Manufacturer Part Number" ""
+			(at 92.71 105.41 0)
+			(effects

Commit message: Update layout, optimize sub-sheet for reusability
Parts:
- added J2: Conn_01x02_Pin, Connector_JST:JST_XH_B2B-XH-A_1x02_P2.50mm_Vertical, symbol Connector:Conn_01x02_Pin
Connections:
- new net BAT+: J2.2 (Pin_2)
- new net BAT-: J2.1 (Pin_1)
Other:
- note added: "Battery Power Port"
- note added: "USB Data Output"
- note removed: "USB Data Lines"
- moved on the sheet: H5, H6, H7, H8
Changed lines of the file:
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@@
 	(rectangle
 		(start 86.36 95.25)
-		(end 138.43 120.65)
+		(end 138.43 127)
 		(stroke
 			(width 0)
@@
 		)
 	)
+	(rectangle
+		(start 138.43 95.25)
+		(end 195.58 127)
+		(stroke
+			(width 0)
+			(type default)
+		)
+		(fill
+			(type none)
+		)
+	)
 	(text "Mounting Holes"
 		(exclude_from_sim no)
@@
 		)
 	)
+	(text "Battery Power Port"
+		(exclude_from_sim no)
+		(at 164.846 99.568 0)
+		(effects
+			(font
+				(size 1.27 1.27)
+			)
+		)
+	)
 	(text "PWR MGR Board specific features"
 		(exclude_from_sim no)
@@
 		)
 	)
-	(text "USB Data Lines"
+	(text "USB Data Output"
 		(exclude_from_sim no)
 		(at 112.268 68.326 0)
@@
 				(size 1.27 1.27)
 			)
+		)
+	)
+	(wire
+		(pts
+			(xy 152.4 113.03) (xy 168.91 113.03)
+		)
+		(stroke
+			(width 0)
+			(type default)
 		)
 	)
@@
 	(wire
 		(pts
+			(xy 152.4 110.49) (xy 168.91 110.49)
+		)
+		(stroke
+			(width 0)
+			(type default)
+		)
+	)
+	(wire
+		(pts
 			(xy 109.22 81.28) (xy 109.22 80.01)
 		)
@@
 		)
 	)
+	(hierarchical_label "BAT+"
+		(shape input)
+		(at 152.4 110.49 180)
+		(effects
+			(font
+				(size 1.27 1.27)
+			)
+			(justify right)
+		)
+	)
+	(hierarchical_label "BAT-"
+		(shape input)
+		(at 152.4 113.03 180)
+		(effects
+			(font
+				(size 1.27 1.27)
+			)
+			(justify right)
+		)
+	)
 	(hierarchical_label "3.3V"
 		(shape input)
-		(at 154.94 78.74 90)
-		(effects
-			(font
-				(size 1.27 1.27)
-			)
-			(justify left)
+		(at 154.94 78.74 180)
+		(effects
+			(font
+				(size 1.27 1.27)
+			)
+			(justify right)
 		)
 	)
@@
 	(symbol
 		(lib_id "Mechanical:MountingHole")
-		(at 116.84 105.41 0)
+		(at 116.84 106.68 0)
 		(unit 1)
 		(exclude_from_sim no)
@@
 		(fields_autoplaced yes)
 		(property "Reference" "H7"
-			(at 119.38 104.1399 0)
+			(at 119.38 105.4099 0)
 			(effects
 				(font
@@
 		)
 		(property "Value" "MountingHole"
-			(at 119.38 106.6799 0)
+			(at 119.38 107.9499 0)
 			(effects
 				(font
@@
 		)
 		(property "Footprint" "MountingHole:MountingHole_2.1mm"
-			(at 116.84 105.41 0)
+			(at 116.84 106.68 0)
 			(effects
 				(font
@@
 		)
 		(property "Datasheet" "~"
-			(at 116.84 105.41 0)
+			(at 116.84 106.68 0)
 			(effects
 				(font
@@
 		)
 		(property "Description" "Mounting Hole without connection"
-			(at 116.84 105.41 0)
+			(at 116.84 106.68 0)
 			(effects
 				(font
@@
 		)
 		(property "Manufacturer Part Number" ""
-			(at 116.84 105.41 0)
+			(at 116.84 106.68 0)
 			(effects
 				(font
@@
 	(symbol
 		(lib_id "Mechanical:MountingHole")
-		(at 92.71 111.76 0)
+		(at 92.71 115.57 0)
 		(unit 1)
 		(exclude_from_sim no)
@@
 		(fields_autoplaced yes)
 		(property "Reference" "H6"
-			(at 95.25 110.4899 0)
+			(at 95.25 114.2999 0)
 			(effects
 				(font
@@
 		)
 		(property "Value" "MountingHole"
-			(at 95.25 113.0299 0)
+			(at 95.25 116.8399 0)
 			(effects
 				(font
@@
 		)
 		(property "Footprint" "MountingHole:MountingHole_2.1mm"
-			(at 92.71 111.76 0)
+			(at 92.71 115.57 0)
 			(effects
 				(font
@@
 		)
 		(property "Datasheet" "~"
-			(at 92.71 111.76 0)
+			(at 92.71 115.57 0)
 			(effects
 				(font
@@
 		)
 		(property "Description" "Mounting Hole without connection"
-			(at 92.71 111.76 0)
+			(at 92.71 115.57 0)
 			(effects
 				(font
@@
 		)
 		(property "Manufacturer Part Number" ""
-			(at 92.71 111.76 0)
+			(at 92.71 115.57 0)
 			(effects
 				(font
@@
 	(symbol
 		(lib_id "Mechanical:MountingHole")
-		(at 116.84 111.76 0)
+		(at 116.84 115.57 0)
 		(unit 1)
 		(exclude_from_sim no)
@@
 		(fields_autoplaced yes)
 		(property "Reference" "H8"
-			(at 119.38 110.4899 0)
+			(at 119.38 114.2999 0)
 			(effects
 				(font
@@
 		)
 		(property "Value" "MountingHole"
-			(at 119.38 113.0299 0)
+			(at 119.38 116.8399 0)
 			(effects
 				(font
@@
 		)
 		(property "Footprint" "MountingHole:MountingHole_2.1mm"
-			(at 116.84 111.76 0)
+			(at 116.84 115.57 0)
 			(effects
 				(font
@@
 		)
 		(property "Datasheet" "~"
-			(at 116.84 111.76 0)
+			(at 116.84 115.57 0)
 			(effects
 				(font
@@
 		)
 		(property "Description" "Mounting Hole without connection"
-			(at 116.84 111.76 0)
+			(at 116.84 115.57 0)
 			(effects
 				(font
@@
 		)
 		(property "Manufacturer Part Number" ""
-			(at 116.84 111.76 0)
+			(at 116.84 115.57 0)
 			(effects
 				(font
@@
 				(path "/16b2e4e2-6399-42b6-a8e6-a11780888710/9a4ce8ea-f122-49e0-9f9a-908eb36e3c79"
 					(reference "H8")
+					(unit 1)
+				)
+			)
+		)
+	)
+	(symbol
+		(lib_id "Connector:Conn_01x02_Pin")
+		(at 173.99 113.03 180)
+		(unit 1)
+		(exclude_from_sim no)
+		(in_bom yes)
+		(on_board yes)
+		(dnp no)
+		(fields_autoplaced yes)
+		(property "Reference" "J2"
+			(at 175.26 110.4899 0)
+			(effects
+				(font
+					(size 1.27 1.27)
+				)
+				(justify right)
+			)
+		)
+		(property "Value" "Conn_01x02_Pin"
+			(at 175.26 113.0299 0)
+			(effects
+				(font
+					(size 1.27 1.27)
+				)
+				(justify right)
+			)
+		)
+		(property "Footprint" "Connector_JST:JST_XH_B2B-XH-A_1x02_P2.50mm_Vertical"
+			(at 173.99 113.03 0)
+			(effects
+				(font
+					(size 1.27 1.27)
+				)
+				(hide yes)
+			)
+		)
+		(property "Datasheet" "~"
+			(at 173.99 113.03 0)
+			(effects
+				(font
+					(size 1.27 1.27)
+				)
+				(hide yes)
+			)
+		)
+		(property "Description" "Generic connector, single row, 01x02, script generated"
+			(at 173.99 113.03 0)
+			(effects
+				(font
+					(size 1.27 1.27)
+				)
+				(hide yes)
+			)
+		)
+		(property "Manufacturer Part Number" " B2B-XH-A"
+			(at 173.99 113.03 0)
+			(effects
+				(font
+					(size 1.27 1.27)
+				)
+				(hide yes)
+			)
+		)
+		(pin "1"
+		)
+		(pin "2"
+		)
+		(instances
+			(project "PWR-MGR-PCB"
+				(path "/16b2e4e2-6399-42b6-a8e6-a11780888710/9a4ce8ea-f122-49e0-9f9a-908eb36e3c79"
+					(reference "J2")
 					(unit 1)
 				)
@@
 	(symbol
 		(lib_id "Mechanical:MountingHole")
-		(at 92.71 105.41 0)
+		(at 92.71 106.68 0)
 		(unit 1)
 		(exclude_from_sim no)
@@
 		(on_board yes)
 		(dnp no)
-		(fields_autoplaced yes)
 		(property "Reference" "H5"
-			(at 95.25 104.1399 0)
+			(at 95.25 105.4099 0)
 			(effects
 				(font
@@
 		)
 		(property "Value" "MountingHole"
-			(at 95.25 106.6799 0)
+			(at 95.25 107.9499 0)
 			(effects
 				(font
@@
 		)
 		(property "Footprint" "MountingHole:MountingHole_2.1mm"
-			(at 92.71 105.41 0)
+			(at 92.71 106.68 0)
 			(effects
 				(font
@@
 		)
 		(property "Datasheet" "~"
-			(at 92.71 105.41 0)
+			(at 92.71 106.68 0)
 			(effects
 				(font
@@
 		)
 		(property "Description" "Mounting Hole without connection"
-			(at 92.71 105.41 0)
+			(at 92.71 106.68 0)
 			(effects
 				(font
@@
 		)
 		(property "Manufacturer Part Number" ""
-			(at 92.71 105.41 0)
-			(effects
-				(font
+			(at 92.71 106.68 0)
+			(effects
+				(font
