File: PWR-MGR-PCB/output.kicad_sch (KiCad schematic)
At the start: 26 parts, among them J10 Conn_01x01_Socket, J11 Conn_01x01_Socket, J12 Conn_01x01_Socket, J13 Conn_01x01_Socket, J14 Conn_01x01_Socket, J15 Conn_01x01_Socket, J16 Conn_01x01_Socket, J17 Conn_01x01_Socket, J18 Conn_01x01_Socket, J19 Conn_01x01_Socket, J20 Conn_01x01_Socket, J21 Conn_01x01_Socket, J22 Conn_01x01_Socket, J23 Conn_01x01_Socket, J24 Conn_01x01_Socket, J26 Conn_01x01_Socket, J27 Conn_01x01_Socket, J5 Conn_01x01_Socket, J6 Conn_01x01_Socket, J7 Conn_01x01_Socket, J8 Conn_01x01_Socket, J9 Conn_01x01_Socket

Commit message: finish routing
Parts:
- renumbered H5 to H1, H6 to H2, H7 to H3, H8 to H4, J6 to J1, J5 to J10, J15 to J11, J16 to J12, J17 to J13, J11 to J14, J12 to J15, J13 to J16, J14 to J17, J7 to J2, J24 to J20, J26 to J21, J27 to J22, J8 to J3, J9 to J4, J10 to J5, J20 to J6, J21 to J7, J22 to J8, J23 to J9
